File: BB_Dash_Display.kicad_pcb (KiCad board)
At the start: 2 copper layers, 54.6 x 71.8 mm, 47 parts, among them J1 Screw_Terminal_01x02, J2 Conn_01x02, J3 Screw_Terminal_01x03, J4 Conn_01x03, J6 Conn_01x40, P8 BeagleBone_Black_Header, P9 BeagleBone_Black_Header, U1 TCAN1042V, U2 STS1024S05, U3 FAN5333B

Commit message: rev a2
Add jumper for can termination
Parts:
- added JP2: Jumper, Connector_PinHeader_2.54mm:PinHeader_1x02_P2.54mm_Horizontal, B.Cu at (88.9, 127.0)
- moved R4 16.6 mm to (87.6, 129.5), turned to 0 degrees
- moved D3 9.92 mm to (114.3, 119.4), turned to 180 degrees
- moved G*** 1.27 mm to (106.7, 95.2)
Connections:
- R4 pad 1: /CANH -> Net-(JP2-Pad2)
Routing:
- net GND: track 124.0 -> 133.1 mm, vias 13 -> 14
- net /LED-: track 46.3 -> 42.4 mm, vias 3 -> 4
- net /LED+: track 41.7 -> 38.2 mm, vias 3 -> 1
- net /CANH: track 90.2 -> 87.1 mm, vias 3 -> 2
- net Net-(JP2-Pad2): track 0.00 -> 2.68 mm
- net /CANL: track 91.1 -> 90.4 mm
Other:
- board text added: "Backlight"
- board text added: "CAN Termination"
- board text added: "Dashboard Display BeagleBone CAN & LCD Version: Rev A2 Designed by: Andrew Chen Date: 2020-03-07"
- board text removed: "Backlight Enable"
- board text removed: "Dashboard Display BeagleBone CAN & LCD Version: Rev A Designed by: Andrew Chen Date: 2020-03-06"

Commit message: rev a3
change to convex resistor arrays
Parts:
- RN1, RN2, RN3, RN4, RN5, RN6, RN7, RN8: footprint Resistor_SMD:R_Array_Concave_4x0603 -> Resistor_SMD:R_Array_Convex_4x0603
Other:
- board text added: "Dashboard Display BeagleBone CAN & LCD Version: Rev A3 Designed by: Andrew Chen Date: 2020-03-07"
- board text removed: "Dashboard Display BeagleBone CAN & LCD Version: Rev A2 Designed by: Andrew Chen Date: 2020-03-07"

Commit message: update schematics for rev b
Parts:
- removed the C1 at (105.4, 101.6)
- removed the C2 at (113.0, 101.6)
- removed the C5 at (110.5, 114.3)
- removed D3: 24V, Diode_SMD:D_SMA
- removed the J1 at (92.4, 92.1)
- removed the J3 at (91.4, 137.2)
- removed J4: Conn_01x03, Connector_Molex:Molex_SPOX_5268-03A_1x03_P2.50mm_Horizontal
- removed JP2: Jumper, Connector_PinHeader_2.54mm:PinHeader_1x02_P2.54mm_Horizontal
- removed the RN5 at (104.1, 125.7)
- removed RN6: 33, Resistor_SMD:R_Array_Convex_4x0603
- removed RN8: 0, Resistor_SMD:R_Array_Convex_4x0603
- removed the U2 at (109.2, 91.4)
- added C10: 22uF, Capacitor_SMD:C_0805_2012Metric, F.Cu at (110.3, 56.1)
- added C11: 22uF, Capacitor_SMD:C_0805_2012Metric, F.Cu at (103.5, 63.9)
- added C3: 10uF, Capacitor_SMD:C_1210_3225Metric, F.Cu at (94.0, 62.2)
- added C4: 220nF, Capacitor_SMD:C_0805_2012Metric, F.Cu at (99.0, 63.9)
- added C7: 0.1uF, Capacitor_SMD:C_0805_2012Metric, F.Cu at (104.6, 60.5)
- added C9: 10uF, Capacitor_SMD:C_1206_3216Metric, F.Cu at (94.0, 66.0)
- added J2: Mini_SPOX, Connector_Molex:Molex_SPOX_5268-03A_1x03_P2.50mm_Horizontal, B.Cu at (113.0, 81.3)
- added L2: 4.7uH, Inductor_SMD:L_Bourns-SRN4018, F.Cu at (94.2, 57.3)
- added R5: 56k, Resistor_SMD:R_0805_2012Metric, F.Cu at (109.1, 60.5)
- added R6: 10k, Resistor_SMD:R_0805_2012Metric, F.Cu at (107.9, 63.5)
- added U1: TPS61165, Package_TO_SOT_SMD:SOT-23-6, F.Cu at (99.8, 60.1)
- C1: renamed from C3; value 10u -> 100nF; footprint Capacitor_SMD:C_1206_3216Metric -> Capacitor_SMD:C_0805_2012Metric
- C2: renamed from C4; value 10u -> 10uF
- C5: renamed from C6; value 100n -> 100nF
- C6: renamed from C7; value 100n -> 100nF
- C8: value 100u -> 10uF; footprint Capacitor_THT:CP_Radial_D5.0mm_P2.50mm -> Capacitor_SMD:C_1206_3216Metric
- D2: renamed from D1; value 16V -> SMF4L15A
- F1: footprint Resistor_THT:R_Axial_DIN0207_L6.3mm_D2.5mm_P10.16mm_Horizontal -> Fuse:Fuseholder_Littelfuse_Nano2_154x
- J1: renamed from J6; value Conn_01x40 -> FH12-40S-0.5SH
- J3: renamed from J2; value Conn_01x02 -> Mini_SPOX
- L1: value 15u -> 22uH; footprint Inductor_SMD:L_1210_3225Metric -> Inductor_SMD:L_Bourns-SRN4018
- R2: renamed from R3; value 8.2 -> 3.3
- U3: value FAN5333B -> TPS562200; footprint Package_TO_SOT_SMD:SOT-23-5 -> Package_TO_SOT_SMD:SOT-23-6
- moved U3 54.2 mm to (105.5, 56.8)
- moved C8 25.2 mm to (100.1, 56.2)
- moved J1 8.13 mm to (101.6, 129.5)
- moved J3 3.17 mm to (83.8, 81.3)
- renumbered D2 to D1, R2 to R1, R1 to R3, RN7 to RN5, TP4 to TP2, TP7 to TP3, TP2 to TP4, TP8 to TP6, TP3 to TP7, TP6 to TP8, U1 to U2
Connections:
- net /L_DE renamed /L_DEN
- net /VIN renamed Net-(F1-Pad2)
- C2 pad 1: Net-(C4-Pad1) -> Net-(C2-Pad1)
- C8 pad 1: /VIN_F -> /V_IN
- D1 pad 2: Net-(D2-Pad2) -> Net-(D1-Pad2)
- D2 pad 1: /VIN_F -> /V_IN
- F1 pad 1: /VIN_F -> /V_IN
- J1 pad 13: /LCD_G0 -> GND
- J1 pad 14: /LCD_G1 -> GND
- J1 pad 21: /LCD_B0 -> GND
- J1 pad 22: /LCD_B1 -> GND
- J1 pad 23: /LCD_B2 -> GND
- J1 pad 5: /LCD_R0 -> GND
- J1 pad 6: /LCD_R1 -> GND
- J1 pad 7: /LCD_R2 -> GND
- JP1 pad 1: +5V -> /V_IN
- JP1 pad 2: Net-(C4-Pad1) -> Net-(C2-Pad1)
- L1 pad 1: Net-(C4-Pad1) -> Net-(C2-Pad1)
- L1 pad 2: Net-(D2-Pad2) -> Net-(D1-Pad2)
- R1 pad 1: Net-(R2-Pad1) -> Net-(R1-Pad1)
- R3 pad 1: /L_DISP -> +3V3
- R3 pad 2: +3V3 -> /L_DISP
- R4 pad 1: Net-(JP2-Pad2) -> /CANH
- RN1 pad 1: /LCD_R0 -> /LCD_R3
- RN1 pad 2: /LCD_R1 -> /LCD_R4
- RN1 pad 3: /LCD_R2 -> /LCD_R5
- RN1 pad 4: /LCD_R3 -> /LCD_R6
- RN1 pad 5: /LCD_D0 -> /LCD_D14
- RN1 pad 6: /LCD_D16 -> /LCD_D13
- RN1 pad 7: /LCD_D18 -> /LCD_D12
- RN1 pad 8: /LCD_D21 -> /LCD_D11
- RN2 pad 1: /LCD_R4 -> /LCD_R7
- RN2 pad 2: /LCD_R5 -> /LCD_G2
- RN2 pad 3: /LCD_R6 -> /LCD_G3
- RN2 pad 4: /LCD_R7 -> /LCD_G4
- RN2 pad 5: /LCD_D4 -> /LCD_D7
- RN2 pad 6: /LCD_D3 -> /LCD_D6
- RN2 pad 7: /LCD_D2 -> /LCD_D5
- RN2 pad 8: /LCD_D1 -> /LCD_D15
- RN3 pad 1: /LCD_G0 -> /LCD_G5
- RN3 pad 2: /LCD_G1 -> /LCD_G6
- RN3 pad 3: /LCD_G2 -> /LCD_G7
- RN3 pad 4: /LCD_G3 -> /LCD_B3
- RN3 pad 5: /LCD_D6 -> /LCD_D0
- RN3 pad 6: /LCD_D5 -> /LCD_D10
- RN3 pad 7: /LCD_D19 -> /LCD_D9
- RN3 pad 8: /LCD_D22 -> /LCD_D8
- RN4 pad 1: /LCD_G4 -> /LCD_B4
- RN4 pad 2: /LCD_G5 -> /LCD_B5
- RN4 pad 3: /LCD_G6 -> /LCD_B6
- RN4 pad 4: /LCD_G7 -> /LCD_B7
- RN4 pad 5: /LCD_D10 -> /LCD_D4
- RN4 pad 6: /LCD_D9 -> /LCD_D3
- RN4 pad 7: /LCD_D8 -> /LCD_D2
- RN4 pad 8: /LCD_D7 -> /LCD_D1
- TP2 pad 1: /VIN_F -> /V_IN
- U2 pad 3: +5V -> +3V3
- U2 pad 5: +3V3 -> +5V
- U3 pad 1: Net-(D2-Pad2) -> GND
- U3 pad 2: GND -> Net-(C7-Pad1)
- U3 pad 3: /LED- -> /V_IN
- U3 pad 4: Net-(R2-Pad1) -> Net-(R5-Pad2)
- U3 pad 5: Net-(C4-Pad1) -> /V_IN
Routing:
- net +3V3: track 140.0 -> 0.00 mm, vias 4 -> 0
- net GND: track 133.1 -> 0.00 mm, vias 14 -> 0
- net /CANL: track 90.4 -> 0.00 mm, vias 3 -> 0
- net /CANH: track 87.1 -> 0.00 mm, vias 2 -> 0
- net +5V: track 78.1 -> 0.00 mm, vias 3 -> 0
- net /LCD_D18: track 72.0 -> 0.00 mm, vias 1 -> 0
- net /LCD_D21: track 71.7 -> 0.00 mm, vias 1 -> 0
- net /LCD_D19: track 67.6 -> 0.00 mm, vias 1 -> 0
- net /LCD_D16: track 66.5 -> 0.00 mm, vias 1 -> 0
- net /LCD_D22: track 63.6 -> 0.00 mm, vias 1 -> 0
- net /LCD_D17: track 55.1 -> 0.00 mm, vias 1 -> 0
- net /LCD_D1: track 51.2 -> 0.00 mm, vias 1 -> 0
- net /LCD_D20: track 51.1 -> 0.00 mm, vias 1 -> 0
- net /LCD_D0: track 49.3 -> 0.00 mm, vias 1 -> 0
- net /LCD_D23: track 49.0 -> 0.00 mm, vias 1 -> 0
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Other:
- board size 54.6 x 71.8 mm -> 54.6 x 61 mm

Commit message: archive stuff
Parts:
- C1, C10, C11, C4, C5, C6, C7: footprint Capacitor_SMD:C_0805_2012Metric -> archive:C_0805_2012Metric
- C2, C8, C9: footprint Capacitor_SMD:C_1206_3216Metric -> archive:C_1206_3216Metric
- C3: footprint Capacitor_SMD:C_1210_3225Metric -> archive:C_1210_3225Metric
- D1, D2: footprint Diode_SMD:D_SOD-123 -> archive:D_SOD-123
- F1: footprint Fuse:Fuseholder_Littelfuse_Nano2_154x -> archive:Fuseholder_Littelfuse_Nano2_154x
- G***: footprint project:OUR-Logo -> archive:OUR-Logo
- J1: footprint Connector_FFC-FPC:Hirose_FH12-40S-0.5SH_1x40-1MP_P0.50mm_Horizontal -> archive:Hirose_FH12-40S-0.5SH_1x40-1MP_P0.50mm_Horizontal
- J2: footprint Connector_Molex:Molex_SPOX_5268-03A_1x03_P2.50mm_Horizontal -> archive:Molex_SPOX_5268-03A_1x03_P2.50mm_Horizontal
- J3: footprint Connector_Molex:Molex_SPOX_5268-02A_1x02_P2.50mm_Horizontal -> archive:Molex_SPOX_5268-02A_1x02_P2.50mm_Horizontal
- JP1: footprint Jumper:SolderJumper-2_P1.3mm_Open_TrianglePad1.0x1.5mm -> archive:SolderJumper-2_P1.3mm_Open_TrianglePad1.0x1.5mm
- L1, L2: footprint Inductor_SMD:L_Bourns-SRN4018 -> archive:L_Bourns-SRN4018
- P8, P9: footprint project:PinHeader_2x23_P2.54mm_Vertical_Flip -> archive:PinHeader_2x23_P2.54mm_Vertical_Flip
- R1, R2, R3, R4, R5, R6: footprint Resistor_SMD:R_0805_2012Metric -> archive:R_0805_2012Metric
- REF**: footprint project:BeagleBone-Black_Flip -> archive:BeagleBone-Black_Flip
- RN1, RN2, RN3, RN4, RN5: footprint Resistor_SMD:R_Array_Convex_4x0603 -> archive:R_Array_Convex_4x0603
- TP1, TP2, TP3, TP4, TP5, TP6, TP7, TP8, TP9: footprint TestPoint:TestPoint_THTPad_D2.0mm_Drill1.0mm -> archive:TestPoint_THTPad_D2.0mm_Drill1.0mm
- U1, U3: footprint Package_TO_SOT_SMD:SOT-23-6 -> archive:SOT-23-6
- U2: footprint Package_SO:SOIC-8_3.9x4.9mm_P1.27mm -> archive:SOIC-8_3.9x4.9mm_P1.27mm

Commit message: rev b
Parts:
- removed G***: LOGO, archive:OUR-Logo
- D2: moved to B.Cu
- moved R4 57.4 mm to (114.3, 78.7), turned to 180 degrees
- moved U1 47.8 mm to (91.4, 107.2), turned to 270 degrees
- moved C4 45.1 mm to (88.4, 107.7), turned to 90 degrees
- moved C3 42.0 mm to (84.3, 103.1), turned to 90 degrees
- moved C8 39.8 mm to (84.8, 93.0), turned to 270 degrees
- moved C5 39.8 mm to (119.4, 91.4)
- moved U3 38.9 mm to (91.9, 93.2)
- moved C10 35.8 mm to (98.0, 89.7), turned to 270 degrees
- moved R5 35.2 mm to (96.0, 93.2), turned to 270 degrees
- moved C7 32.5 mm to (87.9, 88.4), turned to 90 degrees
- moved L2 31.9 mm to (91.9, 89.2)
- moved R6 31.3 mm to (98.0, 93.2), turned to 90 degrees
- moved U2 31.0 mm to (114.3, 91.4)
- moved JP1 27.9 mm to (91.4, 98.0), turned to 0 degrees
- moved C9 27.7 mm to (87.4, 93.0), turned to 270 degrees
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Connections:
- J1 pad MP: GND -> Net-(J1-PadMP)
Routing:
- net GND: track 0.00 -> 182.8 mm, vias 0 -> 15
- net +3V3: track 0.00 -> 78.5 mm, vias 0 -> 3
- net /LED+: track 0.00 -> 61.6 mm, vias 0 -> 1
- net +5V: track 0.00 -> 61.3 mm, vias 0 -> 2
- net /V_IN: track 0.00 -> 53.7 mm, vias 0 -> 2
- net /LED-: track 0.00 -> 46.2 mm, vias 0 -> 1
- net /LCD_D11: track 0.00 -> 41.6 mm, vias 0 -> 1
- net /EHRPWM1A: track 0.00 -> 40.4 mm, vias 0 -> 2
- net /LCD_D15: track 0.00 -> 39.9 mm, vias 0 -> 1
- net /LCD_D12: track 0.00 -> 37.5 mm, vias 0 -> 1
- net /LCD_D13: track 0.00 -> 36.7 mm, vias 0 -> 1
- net /LCD_D14: track 0.00 -> 36.7 mm, vias 0 -> 1
- net /LCD_D5: track 0.00 -> 35.9 mm, vias 0 -> 1
- net /LCD_D7: track 0.00 -> 34.8 mm, vias 0 -> 1
- net /LCD_D9: track 0.00 -> 33.0 mm, vias 0 -> 1
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Other:
- net class Default: clearance 0.1524 -> 0.2; trace_width 0.1524 -> 0.2
- rule trace_clearance: 0.1524 -> 0.2
- board text added: "BL+"
- board text added: "BL-"
- board text added: "Dashboard Display BeagleBone CAN & LCD Version: Rev B Designed by: Andrew Chen Date: 2020-06-02"
- board text added: "VIN"
- board text removed: "CAN Termination"
- board text removed: "Dashboard Display BeagleBone CAN & LCD Version: Rev A3 Designed by: Andrew Chen Date: 2020-03-07"
- board text removed: "LED+"
- board text removed: "LED-"
- board text removed: "Vin"
