File: BB_Dash_Display.sch (KiCad schematic (older format))
At the start: 45 parts, among them J1 Screw_Terminal_01x02, J2 Conn_01x02, J3 Screw_Terminal_01x03, J4 Conn_01x03, J6 Conn_01x40, P8 BeagleBone_Black_Header, P9 BeagleBone_Black_Header, U1 TCAN1042V, U2 STS1024S05, U3 FAN5333B

Commit message: rev a2
Add jumper for can termination
Parts:
- added JP2: Jumper, Connector_PinHeader_2.54mm:PinHeader_1x02_P2.54mm_Horizontal, symbol Device:Jumper
Connections:
- net CANH: now also JP2.1; no longer R4.1
- new net: JP2.2, R4.1
Other:
- moved on the sheet: R4
Changed lines of the file:
@@
 Sheet 1 1
 Title "Dashboard Display BeagleBone CAN & LCD"
-Date ""
-Rev "A"
+Date "2020-03-07"
+Rev "A2"
 Comp ""
 Comment1 ""
@@
 L Device:R_Small R4
 U 1 1 5F2009F0
-P 4900 6900
-F 0 "R4" H 4959 6946 50  0000 L CNN
-F 1 "120" H 4959 6855 50  0000 L CNN
-F 2 "Resistor_SMD:R_0805_2012Metric" H 4900 6900 50  0001 C CNN
-F 3 "~" H 4900 6900 50  0001 C CNN
-F 4 "RC0805FR-07120RL" H 4900 6900 50  0001 C CNN "Part"
-	1    4900 6900
+P 5500 6900
+F 0 "R4" H 5559 6946 50  0000 L CNN
+F 1 "120" H 5559 6855 50  0000 L CNN
+F 2 "Resistor_SMD:R_0805_2012Metric" H 5500 6900 50  0001 C CNN
+F 3 "~" H 5500 6900 50  0001 C CNN
+F 4 "RC0805FR-07120RL" H 5500 6900 50  0001 C CNN "Part"
+	1    5500 6900
 	1    0    0    -1
 $EndComp
 Wire Wire Line
 	4500 6800 4900 6800
-Wire Wire Line
-	4500 7000 4900 7000
 $Comp
 L project:R_Pack04 RN1
@@
 Wire Wire Line
 	2600 4500 3000 4500
+$Comp
+L Device:Jumper JP2
+U 1 1 5E679252
+P 5200 6800
+F 0 "JP2" H 5200 6973 50  0000 C CNN
+F 1 "Jumper" H 5200 6973 50  0001 C CNN
+F 2 "Connector_PinHeader_2.54mm:PinHeader_1x02_P2.54mm_Horizontal" H 5200 6800 50  0001 C CNN
+F 3 "~" H 5200 6800 50  0001 C CNN
+	1    5200 6800
+	1    0    0    -1
+$EndComp
+Wire Wire Line
+	4500 7000 5500 7000
 $EndSCHEMATC

Commit message: rev a3
change to convex resistor arrays
Parts:
- J4: Part 22057025 -> 22057035
- RN1, RN2, RN3, RN4, RN5, RN6, RN7, RN8: footprint Resistor_SMD:R_Array_Concave_4x0603 -> Resistor_SMD:R_Array_Convex_4x0603
Changed lines of the file:
@@
 Title "Dashboard Display BeagleBone CAN & LCD"
 Date "2020-03-07"
-Rev "A2"
+Rev "A3"
 Comp ""
 Comment1 ""
@@
 F 2 "Connector_Molex:Molex_SPOX_5268-03A_1x03_P2.50mm_Horizontal" H 2000 6700 50  0001 C CNN
 F 3 "~" H 2000 6700 50  0001 C CNN
-F 4 "22057025" H 2000 6700 50  0001 C CNN "Part"
+F 4 "22057035" H 2000 6700 50  0001 C CNN "Part"
 	1    2000 6700
 	1    0    0    -1
@@
 F 0 "RN1" V 6400 1700 50  0000 C CNN
 F 1 "33" V 6400 1350 50  0000 C CNN
-F 2 "Resistor_SMD:R_Array_Concave_4x0603" V 6925 1500 50  0001 C CNN
+F 2 "Resistor_SMD:R_Array_Convex_4x0603" V 6925 1500 50  0001 C CNN
 F 3 "~" H 6650 1500 50  0001 C CNN
 F 4 "YC164-JR-0733RL" H 6650 1500 50  0001 C CNN "Part"
@@
 F 0 "RN2" V 6400 2100 50  0000 C CNN
 F 1 "33" V 6400 1750 50  0000 C CNN
-F 2 "Resistor_SMD:R_Array_Concave_4x0603" V 6925 1900 50  0001 C CNN
+F 2 "Resistor_SMD:R_Array_Convex_4x0603" V 6925 1900 50  0001 C CNN
 F 3 "~" H 6650 1900 50  0001 C CNN
 F 4 "YC164-JR-0733RL" H 6650 1900 50  0001 C CNN "Part"
@@
 F 0 "RN3" V 6400 2500 50  0000 C CNN
 F 1 "33" V 6400 2150 50  0000 C CNN
-F 2 "Resistor_SMD:R_Array_Concave_4x0603" V 6925 2300 50  0001 C CNN
+F 2 "Resistor_SMD:R_Array_Convex_4x0603" V 6925 2300 50  0001 C CNN
 F 3 "~" H 6650 2300 50  0001 C CNN
 F 4 "YC164-JR-0733RL" H 6650 2300 50  0001 C CNN "Part"
@@
 F 0 "RN4" V 6400 2900 50  0000 C CNN
 F 1 "33" V 6400 2550 50  0000 C CNN
-F 2 "Resistor_SMD:R_Array_Concave_4x0603" V 6925 2700 50  0001 C CNN
+F 2 "Resistor_SMD:R_Array_Convex_4x0603" V 6925 2700 50  0001 C CNN
 F 3 "~" H 6650 2700 50  0001 C CNN
 F 4 "YC164-JR-0733RL" H 6650 2700 50  0001 C CNN "Part"
@@
 F 0 "RN5" V 6400 3300 50  0000 C CNN
 F 1 "33" V 6400 2950 50  0000 C CNN
-F 2 "Resistor_SMD:R_Array_Concave_4x0603" V 6925 3100 50  0001 C CNN
+F 2 "Resistor_SMD:R_Array_Convex_4x0603" V 6925 3100 50  0001 C CNN
 F 3 "~" H 6650 3100 50  0001 C CNN
 F 4 "YC164-JR-0733RL" H 6650 3100 50  0001 C CNN "Part"
@@
 F 0 "RN6" V 6400 3700 50  0000 C CNN
 F 1 "33" V 6400 3350 50  0000 C CNN
-F 2 "Resistor_SMD:R_Array_Concave_4x0603" V 6925 3500 50  0001 C CNN
+F 2 "Resistor_SMD:R_Array_Convex_4x0603" V 6925 3500 50  0001 C CNN
 F 3 "~" H 6650 3500 50  0001 C CNN
 F 4 "YC164-JR-0733RL" H 6650 3500 50  0001 C CNN "Part"
@@
 U 1 1 5F2F466B
 P 6650 4050
-F 0 "RN7" V 6400 4250 50  0000 C CNN
+F 0 "RN7" V 6350 4050 50  0000 C CNN
 F 1 "33" V 6400 3900 50  0000 C CNN
-F 2 "Resistor_SMD:R_Array_Concave_4x0603" V 6925 4050 50  0001 C CNN
+F 2 "Resistor_SMD:R_Array_Convex_4x0603" V 6925 4050 50  0001 C CNN
 F 3 "~" H 6650 4050 50  0001 C CNN
 F 4 "YC164-JR-0733RL" H 6650 4050 50  0001 C CNN "Part"
@@
 U 1 1 5F2F4EA2
 P 6650 4700
-F 0 "RN8" V 6400 4900 50  0000 C CNN
+F 0 "RN8" V 6350 4700 50  0000 C CNN
 F 1 "0" V 6400 4550 50  0000 C CNN
-F 2 "Resistor_SMD:R_Array_Concave_4x0603" V 6925 4700 50  0001 C CNN
+F 2 "Resistor_SMD:R_Array_Convex_4x0603" V 6925 4700 50  0001 C CNN
 F 3 "~" H 6650 4700 50  0001 C CNN
 F 4 "YC164-JR-070RL" H 6650 4700 50  0001 C CNN "Part"

Commit message: update schematics for rev b
Parts:
- removed C1, C2: 10u, Capacitor_SMD:C_1206_3216Metric, symbol Device:C_Small
- removed C5: 10u, Capacitor_SMD:C_1206_3216Metric, symbol Device:C
- removed C8: 100u, Capacitor_THT:CP_Radial_D5.0mm_P2.50mm, symbol Device:CP_Small
- removed D3: 24V, Diode_SMD:D_SMA, symbol Device:D_Zener
- removed J1: Screw_Terminal_01x02, TerminalBlock_Phoenix:TerminalBlock_Phoenix_PT-1,5-2-3.5-H_1x02_P3.50mm_Horizontal, symbol Connector:Screw_Terminal_01x02
- removed J3: Screw_Terminal_01x03, TerminalBlock_Phoenix:TerminalBlock_Phoenix_PT-1,5-3-3.5-H_1x03_P3.50mm_Horizontal, symbol Connector:Screw_Terminal_01x03
- removed JP2: Jumper, Connector_PinHeader_2.54mm:PinHeader_1x02_P2.54mm_Horizontal, symbol Device:Jumper
- removed RN5, RN6: 33, Resistor_SMD:R_Array_Convex_4x0603, symbol project:R_Pack04
- removed RN8: 0, Resistor_SMD:R_Array_Convex_4x0603, symbol project:R_Pack04
- removed U2: STS1024S05, project:STS1024S05, symbol project:STS1024S05
- removed U3: FAN5333B, Package_TO_SOT_SMD:SOT-23-5, symbol project:FAN5333
- added C10, C11: 22uF, Capacitor_SMD:C_0805_2012Metric, symbol Device:C
- added C3: 10uF, Capacitor_SMD:C_1210_3225Metric, symbol Device:C_Small
- added C4: 220nF, Capacitor_SMD:C_0805_2012Metric, symbol Device:C_Small
- added C7: 0.1uF, Capacitor_SMD:C_0805_2012Metric, symbol Device:C_Small
- added C8, C9: 10uF, Capacitor_SMD:C_1206_3216Metric, symbol Device:C
- added L2: 4.7uH, Inductor_SMD:L_Bourns-SRN4018, symbol Device:L
- added R5: 56k, Resistor_SMD:R_0805_2012Metric, symbol Device:R_Small
- added R6: 10k, Resistor_SMD:R_0805_2012Metric, symbol Device:R_Small
- added U1: TPS61165, Package_TO_SOT_SMD:SOT-23-6, symbol project:TPS61165
- added U3: TPS562200, Package_TO_SOT_SMD:SOT-23-6, symbol Regulator_Switching:TPS562200
- C1: renamed from C3; value 10u -> 100nF; footprint Capacitor_SMD:C_1206_3216Metric -> Capacitor_SMD:C_0805_2012Metric; Part GRM31CR71E106KA12 -> (none)
- C2: renamed from C4; value 10u -> 10uF; symbol Device:C -> Device:C_Small; Comment (none) -> 25V; Part GRM31CR71E106KA12 -> (none); Voltage (none) -> 25V
- C5: renamed from C6; value 100n -> 100nF; Part GRM21B7U1A104JA01L -> (none)
- C6: renamed from C7; value 100n -> 100nF; Part GRM21B7U1A104JA01L -> (none)
- D2: renamed from D1; value 16V -> SMF4L15A; symbol Device:D_Schottky_Small -> Device:D_Zener
- F1: footprint Resistor_THT:R_Axial_DIN0207_L6.3mm_D2.5mm_P10.16mm_Horizontal -> Fuse:Fuseholder_Littelfuse_Nano2_154x; Part 0251001. -> 154001.0
- J1: renamed from J6; value Conn_01x40 -> FH12-40S-0.5SH
- J2: renamed from J4; value Conn_01x03 -> Mini_SPOX
- J3: renamed from J2; value Conn_01x02 -> Mini_SPOX
- L1: value 15u -> 22uH; footprint Inductor_SMD:L_1210_3225Metric -> Inductor_SMD:L_Bourns-SRN4018; Part BRL3225T150K -> SRN4018-220M
- R1: renamed from R2; Part RC0805FR-0733RL -> (none)
- R2: renamed from R3; value 8.2 -> 3.3; Part RC0805FR-078R2L -> (none)
- R3: renamed from R1; Part RC0805FR-0733RL -> (none)
- R4: DNP (none) -> DNP; Part RC0805FR-07120RL -> 120Ω 0805
- renumbered D2 to D1, RN7 to RN5, TP4 to TP2, TP7 to TP3, TP2 to TP4, TP8 to TP6, TP3 to TP7, TP6 to TP8, U1 to U2
Connections:
- net LCD_B0 is gone; now on net GND: J1.21 (Pin_21)
- net LCD_B1 is gone; now on net GND: J1.22 (Pin_22)
- net LCD_B2 is gone; now on net GND: J1.23 (Pin_23)
- net +3V3: now also R3.1, U2.3 (VCC); no longer R3.2
- net +5V: now also U2.5 (VIO), C10.1, C11.1, L2.2, R5.1; no longer JP1.1 (A)
- net CANH: now also R4.1, U2.7 (CANH)
- net CANL: now also U2.6 (CANL)
- net DCAN1_RX: now also U2.4 (RXD)
- net DCAN1_TX: now also U2.1 (TXD)
- net GND: now also J1.13 (Pin_13), J1.14 (Pin_14), J1.5 (Pin_5), J1.6 (Pin_6), J1.7 (Pin_7), U2.2 (GND), U2.8 (STB), C10.2, C11.2, C3.2, C4.2, C8.2, C9.2, R6.2, U1.4 (GND), U3.1 (GND)
- net LCD_B3: now also RN3.4 (R4.1)
- net LCD_B4: now also RN4.1 (R1.1)
- net LCD_B5: now also RN4.2 (R2.1)
- net LCD_B6: now also RN4.3 (R3.1)
- net LCD_B7: now also RN4.4 (R4.1)
- net LCD_D0: now also RN3.5 (R4.2); no longer RN1.5 (R4.2)
- net LCD_D1: now also RN4.8 (R1.2); no longer RN2.8 (R1.2)
- net LCD_D10: now also RN3.6 (R3.2); no longer RN4.5 (R4.2)
- net LCD_D11: now also RN1.8 (R1.2)
- net LCD_D12: now also RN1.7 (R2.2)
- net LCD_D13: now also RN1.6 (R3.2)
- net LCD_D14: now also RN1.5 (R4.2)
- net LCD_D15: now also RN2.8 (R1.2)
- net LCD_D16: no longer RN1.6 (R3.2)
- net LCD_D18: no longer RN1.7 (R2.2)
- net LCD_D19: no longer RN3.7 (R2.2)
- net LCD_D2: now also RN4.7 (R2.2); no longer RN2.7 (R2.2)
- net LCD_D21: no longer RN1.8 (R1.2)
- net LCD_D22: no longer RN3.8 (R1.2)
- net LCD_D3: now also RN4.6 (R3.2); no longer RN2.6 (R3.2)
- net LCD_D4: now also RN4.5 (R4.2); no longer RN2.5 (R4.2)
- net LCD_D5: now also RN2.7 (R2.2); no longer RN3.6 (R3.2)
- net LCD_D6: now also RN2.6 (R3.2); no longer RN3.5 (R4.2)
- net LCD_D7: now also RN2.5 (R4.2); no longer RN4.8 (R1.2)
- net LCD_D8: now also RN3.8 (R1.2); no longer RN4.7 (R2.2)
- net LCD_D9: now also RN3.7 (R2.2); no longer RN4.6 (R3.2)
- net LCD_G2: now also RN2.2 (R2.1); no longer RN3.3 (R3.1)
- net LCD_G3: now also RN2.3 (R3.1); no longer RN3.4 (R4.1)
- net LCD_G4: now also RN2.4 (R4.1); no longer RN4.1 (R1.1)
- net LCD_G5: now also RN3.1 (R1.1); no longer RN4.2 (R2.1)
- net LCD_G6: now also RN3.2 (R2.1); no longer RN4.3 (R3.1)
- net LCD_G7: now also RN3.3 (R3.1); no longer RN4.4 (R4.1)
- net LCD_R3: now also RN1.1 (R1.1); no longer RN1.4 (R4.1)
- net LCD_R4: now also RN1.2 (R2.1); no longer RN2.1 (R1.1)
- net LCD_R5: now also RN1.3 (R3.1); no longer RN2.2 (R2.1)
- net LCD_R6: now also RN1.4 (R4.1); no longer RN2.3 (R3.1)
- net LCD_R7: now also RN2.1 (R1.1); no longer RN2.4 (R4.1)
- net LED+: now also C3.1
- net LED-: now also U1.6 (FB)
- net L_DISP: now also R3.2; no longer R3.1
- net at C2.1, JP1.2 (B), L1.1: now also U1.1 (VIN)
- net at D1.2 (A), L1.2: now also U1.3 (SW)
- net at R1.1: now also U1.2 (CTRL)
- removed net LCD_G0: J1.13 (Pin_13), RN3.1 (R1.1)
- removed net LCD_G1: J1.14 (Pin_14), RN3.2 (R2.1)
- removed net LCD_R0: J1.5 (Pin_5), RN1.1 (R1.1)
- removed net LCD_R1: J1.6 (Pin_6), RN1.2 (R2.1)
- removed net LCD_R2: J1.7 (Pin_7), RN1.3 (R3.1)
- net L_DE renamed L_DEN
- net VIN: no longer names the net of F1.2, J3.1 (Pin_1)
- net VIN_F renamed V_IN
- net V_IN: now also JP1.1 (A), C8.1, C9.1, U3.3 (VIN), U3.5 (EN)
- new net: C4.1, U1.5 (COMP)
- new net: C7.1, L2.1, U3.2 (SW)
- new net: R5.2, R6.1, U3.4 (VFB)
- new net: C7.2, U3.6 (VBST)
- no-connect marks 46 -> 62
Other:
- moved on the sheet: C1, C2, C5, C6, D1, D2, F1, J1, J2, J3, JP1, L1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

Commit message: archive stuff
Parts:
- C1, C4, C5, C6, C7: footprint Capacitor_SMD:C_0805_2012Metric -> archive:C_0805_2012Metric; symbol Device:C_Small -> archive:Device_C_Small
- C10, C11: footprint Capacitor_SMD:C_0805_2012Metric -> archive:C_0805_2012Metric; symbol Device:C -> archive:Device_C
- C2: footprint Capacitor_SMD:C_1206_3216Metric -> archive:C_1206_3216Metric; symbol Device:C_Small -> archive:Device_C_Small
- C3: footprint Capacitor_SMD:C_1210_3225Metric -> archive:C_1210_3225Metric; symbol Device:C_Small -> archive:Device_C_Small
- C8, C9: footprint Capacitor_SMD:C_1206_3216Metric -> archive:C_1206_3216Metric; symbol Device:C -> archive:Device_C
- D1: footprint Diode_SMD:D_SOD-123 -> archive:D_SOD-123; symbol Device:D_Schottky -> archive:Device_D_Schottky
- D2: footprint Diode_SMD:D_SOD-123 -> archive:D_SOD-123; symbol Device:D_Zener -> archive:Device_D_Zener
- F1: footprint Fuse:Fuseholder_Littelfuse_Nano2_154x -> archive:Fuseholder_Littelfuse_Nano2_154x; symbol Device:Fuse -> archive:Device_Fuse
- J1: footprint Connector_FFC-FPC:Hirose_FH12-40S-0.5SH_1x40-1MP_P0.50mm_Horizontal -> archive:Hirose_FH12-40S-0.5SH_1x40-1MP_P0.50mm_Horizontal; symbol Connector_Generic_MountingPin:Conn_01x40_MountingPin -> archive:Connector_Generic_MountingPin_Conn_01x40_MountingPin
- J2: footprint Connector_Molex:Molex_SPOX_5268-03A_1x03_P2.50mm_Horizontal -> archive:Molex_SPOX_5268-03A_1x03_P2.50mm_Horizontal; symbol Connector_Generic:Conn_01x03 -> archive:Connector_Generic_Conn_01x03
- J3: footprint Connector_Molex:Molex_SPOX_5268-02A_1x02_P2.50mm_Horizontal -> archive:Molex_SPOX_5268-02A_1x02_P2.50mm_Horizontal; symbol Connector_Generic:Conn_01x02 -> archive:Connector_Generic_Conn_01x02
- JP1: footprint Jumper:SolderJumper-2_P1.3mm_Open_TrianglePad1.0x1.5mm -> archive:SolderJumper-2_P1.3mm_Open_TrianglePad1.0x1.5mm; symbol Jumper:SolderJumper_2_Open -> archive:Jumper_SolderJumper_2_Open
- L1, L2: footprint Inductor_SMD:L_Bourns-SRN4018 -> archive:L_Bourns-SRN4018; symbol Device:L -> archive:Device_L
- P8, P9: footprint project:PinHeader_2x23_P2.54mm_Vertical_Flip -> archive:PinHeader_2x23_P2.54mm_Vertical_Flip; symbol Connector_Generic:Conn_02x23_Odd_Even -> archive:Connector_Generic_Conn_02x23_Odd_Even
- R1, R2, R3, R4, R5, R6: footprint Resistor_SMD:R_0805_2012Metric -> archive:R_0805_2012Metric; symbol Device:R_Small -> archive:Device_R_Small
- RN1, RN2, RN3, RN4, RN5: footprint Resistor_SMD:R_Array_Convex_4x0603 -> archive:R_Array_Convex_4x0603; symbol project:R_Pack04 -> archive:project_R_Pack04
- TP1, TP2, TP3, TP4, TP5, TP6, TP7, TP8, TP9: footprint TestPoint:TestPoint_THTPad_D2.0mm_Drill1.0mm -> archive:TestPoint_THTPad_D2.0mm_Drill1.0mm; symbol Connector:TestPoint -> archive:Connector_TestPoint
- U1: footprint Package_TO_SOT_SMD:SOT-23-6 -> archive:SOT-23-6; symbol project:TPS61165 -> archive:project_TPS61165
- U2: footprint Package_SO:SOIC-8_3.9x4.9mm_P1.27mm -> archive:SOIC-8_3.9x4.9mm_P1.27mm; symbol project:TCAN1042 -> archive:project_TCAN1042
- U3: footprint Package_TO_SOT_SMD:SOT-23-6 -> archive:SOT-23-6; symbol Regulator_Switching:TPS562200 -> archive:Regulator_Switching_TPS562200

Commit message: rev b
Connections:
- net GND: no longer J1.MP (MountPin)
- no-connect marks 62 -> 63
